Commit message: Add power limit and update torque limits

File: legged_examples/legged_unitree/legged_unitree_description/urdf/go1/robot.xacro (robot description, xacro)
@@ -1,14 +1,15 @@
 <?xml version="1.0"?>
 <robot name="go1" xmlns:xacro="http://www.ros.org/wiki/xacro">
-    <xacro:arg name="DEBUG" default="false"/>
-    <xacro:include filename="$(find legged_unitree_description)/urdf/go1/const.xacro"/>
-    <xacro:include filename="$(find legged_unitree_description)/urdf/go1/materials.xacro"/>
-    <xacro:include filename="$(find legged_unitree_description)/urdf/go1/leg.xacro"/>
-    <xacro:include filename="$(find legged_unitree_description)/urdf/go1/gazebo.xacro"/>
-    <xacro:include filename="$(find legged_unitree_description)/urdf/go1/depthCamera.xacro"/>
-    <xacro:include filename="$(find legged_unitree_description)/urdf/go1/ultraSound.xacro"/>
-    <xacro:include filename="$(find legged_unitree_description)/urdf/go1/imu.xacro"/>
+    <xacro:arg name="DEBUG" default="false" />
+    <xacro:include filename="$(find legged_unitree_description)/urdf/go1/const.xacro" />
+    <xacro:include filename="$(find legged_unitree_description)/urdf/go1/materials.xacro" />
+    <xacro:include filename="$(find legged_unitree_description)/urdf/go1/leg.xacro" />
+    <xacro:include filename="$(find legged_unitree_description)/urdf/go1/gazebo.xacro" />
+    <xacro:include filename="$(find legged_unitree_description)/urdf/go1/depthCamera.xacro" />
+    <xacro:include filename="$(find legged_unitree_description)/urdf/go1/ultraSound.xacro" />
+    <xacro:include filename="$(find legged_unitree_description)/urdf/go1/imu.xacro" />
     <!-- Rotor related joint and link is only for demonstrate location. -->
-    <!-- Actually, the rotor will rotate and the joint is not fixed. Reduction ratio should be considered. -->
+    <!-- Actually, the rotor will rotate and the joint is not fixed. Reduction ratio should be
+    considered. -->
     <!-- Debug mode will hung up the robot, use "true" or "false" to switch it. -->
     <!-- <xacro:if value="$(arg DEBUG)">
@@ -35,67 +36,73 @@
     <link name="base">
         <visual>
-            <origin rpy="0 0 0" xyz="0 0 0"/>
+            <origin rpy="0 0 0" xyz="0 0 0" />
             <geometry>
-                <mesh filename="package://legged_unitree_description/meshes/go1/trunk.dae" scale="1 1 1"/>
+                <mesh filename="package://legged_unitree_description/meshes/go1/trunk.dae"
+                    scale="1 1 1" />
             </geometry>
             <!-- <material name="orange"/> -->
         </visual>
         <collision>
-            <origin rpy="0 0 0" xyz="0 0 0"/>
+            <origin rpy="0 0 0" xyz="0 0 0" />
             <geometry>
-                <box size="${trunk_length} ${trunk_width} ${trunk_height}"/>
+                <box size="${trunk_length} ${trunk_width} ${trunk_height}" />
             </geometry>
         </collision>
         <inertial>
-            <origin rpy="0 0 0" xyz="${trunk_com_x} ${trunk_com_y} ${trunk_com_z}"/>
-            <mass value="${trunk_mass}"/>
+            <origin rpy="0 0 0" xyz="${trunk_com_x} ${trunk_com_y} ${trunk_com_z}" />
+            <mass value="${trunk_mass}" />
             <inertia
                 ixx="${trunk_ixx}" ixy="${trunk_ixy}" ixz="${trunk_ixz}"
                 iyy="${trunk_iyy}" iyz="${trunk_iyz}"
-                izz="${trunk_izz}"/>
+                izz="${trunk_izz}" />
         </inertial>
     </link>
-    <xacro:IMU connected_to="base" imu_name="unitree_imu" xyz="0. 0. 0." rpy="0. 0. 0."/>
-    <xacro:leg name="RF" mirror="-1" mirror_dae= "False" front_hind="1"  front_hind_dae="True"  />
-    <xacro:leg name="LF" mirror="1"  mirror_dae="True"   front_hind="1"  front_hind_dae="True"  />
-    <xacro:leg name="RH" mirror="-1" mirror_dae="False"  front_hind="-1" front_hind_dae="False" />
-    <xacro:leg name="LH" mirror="1"  mirror_dae="True"   front_hind="-1" front_hind_dae="False" />
+    <!-- <link name="world" />
+    <joint name="base_world" type="fixed">
+        <parent link="world" />
+        <child link="base" />
+    </joint> -->
+    <xacro:IMU connected_to="base" imu_name="unitree_imu" xyz="0. 0. 0." rpy="0. 0. 0." />
+    <xacro:leg name="RF" mirror="-1" mirror_dae="False" front_hind="1" front_hind_dae="True" />
+    <xacro:leg name="LF" mirror="1" mirror_dae="True" front_hind="1" front_hind_dae="True" />
+    <xacro:leg name="RH" mirror="-1" mirror_dae="False" front_hind="-1" front_hind_dae="False" />
+    <xacro:leg name="LH" mirror="1" mirror_dae="True" front_hind="-1" front_hind_dae="False" />
     <xacro:depthCamera camID="1" name="face">
-        <origin rpy="${PI} 0 0" xyz="0.2785 0.0125 0.0167"/>
+        <origin rpy="${PI} 0 0" xyz="0.2785 0.0125 0.0167" />
     </xacro:depthCamera>
     <xacro:depthCamera camID="2" name="chin">
-        <origin rpy="${PI} ${PI/2} 0" xyz="0.2522 0.0125 -0.0436"/>
+        <origin rpy="${PI} ${PI/2} 0" xyz="0.2522 0.0125 -0.0436" />
     </xacro:depthCamera>
     <xacro:depthCamera camID="3" name="left">
-        <origin rpy="${PI} 0.2618 ${PI/2}" xyz="-0.066 0.082 -0.0176"/>
+        <origin rpy="${PI} 0.2618 ${PI/2}" xyz="-0.066 0.082 -0.0176" />
     </xacro:depthCamera>
     <xacro:depthCamera camID="4" name="right">
-        <origin rpy="${PI} 0.2618 ${-PI/2}" xyz="-0.041 -0.082 -0.0176"/>
+        <origin rpy="${PI} 0.2618 ${-PI/2}" xyz="-0.041 -0.082 -0.0176" />
     </xacro:depthCamera>
     <xacro:depthCamera camID="5" name="rearDown">
-        <origin rpy="${PI} ${PI/2} 0" xyz="-0.0825 0.0125 -0.04365"/>
+        <origin rpy="${PI} ${PI/2} 0" xyz="-0.0825 0.0125 -0.04365" />
     </xacro:depthCamera>
     <joint name="camera_laserscan_joint_left" type="fixed">
-        <origin rpy="0 0.2618 0" xyz="0 0 0"/>
-        <parent link="camera_left"/>
-        <child link="camera_laserscan_link_left"/>
+        <origin rpy="0 0.2618 0" xyz="0 0 0" />
+        <parent link="camera_left" />
+        <child link="camera_laserscan_link_left" />
     </joint>
     <link name="camera_laserscan_link_left">
     </link>
     <joint name="camera_laserscan_joint_right" type="fixed">
-        <origin rpy="0 0.2618 0" xyz="0 0 0"/>
-        <parent link="camera_right"/>
-        <child link="camera_laserscan_link_right"/>
+        <origin rpy="0 0.2618 0" xyz="0 0 0" />
+        <parent link="camera_right" />
+        <child link="camera_laserscan_link_right" />
     </joint>
     <link name="camera_laserscan_link_right">
     </link>
     <xacro:ultraSound name="left">
-        <origin rpy="0 0.2618 ${PI/2}" xyz="-0.0535  0.0826 0.00868"/>
+        <origin rpy="0 0.2618 ${PI/2}" xyz="-0.0535  0.0826 0.00868" />
     </xacro:ultraSound>
     <xacro:ultraSound name="right">
-        <origin rpy="0 0.2618 ${-PI/2}" xyz="-0.0535 -0.0826 0.00868"/>
+        <origin rpy="0 0.2618 ${-PI/2}" xyz="-0.0535 -0.0826 0.00868" />
     </xacro:ultraSound>
     <xacro:ultraSound name="face">
-        <origin rpy="0 0 0" xyz="0.2747 0.0 -0.0088"/>
+        <origin rpy="0 0 0" xyz="0.2747 0.0 -0.0088" />
     </xacro:ultraSound>
 </robot>
